File: IRP PCB/IRP.kicad_pcb (KiCad board)
At the start: 2 copper layers, 18 parts, among them K1 Relay, K2 Relay, Q1 TIP122, Q2 TIP122, U1 LM7805_TO220, U2 ATMEGA328-PU, Y1 Crystal

Commit message: PCB
Parts:
- moved C2 119.3 mm to (54.8, 94.9)
- moved C1 109.9 mm to (58.8, 82.6), turned to 270 degrees
- moved Y1 90.4 mm to (64.3, 95.6), turned to 270 degrees
- moved FTDI1 82.2 mm to (70.0, 92.8), turned to 90 degrees
- moved Battary1 76.6 mm to (61.2, 63.1)
- moved BT1 41.6 mm to (90.2, 76.4), turned to 90 degrees
- moved K1 30.2 mm to (44.2, 113.1)
- moved D2 30.2 mm to (48.3, 106.5)
- moved D1 28.3 mm to (48.1, 82.9)
- moved Motor1 28.3 mm to (36.6, 100.6)
- moved K2 28.3 mm to (44.8, 76.8)
- moved R3 24.3 mm to (73.1, 56.0), turned to 270 degrees
- moved R2 17.6 mm to (65.4, 110.2), turned to 270 degrees
- moved U2 16.9 mm to (77.0, 77.2)
- moved Q1 15.1 mm to (56.6, 115.7)
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Routing:
- net GND: track 174.2 -> 283.5 mm
- net +5V: track 0.00 -> 74.5 mm
- net /TX: track 0.00 -> 45.0 mm
- net /HB2: track 6.27 -> 39.6 mm
- net +12V: track 141.0 -> 111.8 mm
- net /HB1: track 4.89 -> 31.7 mm
- net /RX: track 0.00 -> 26.2 mm
- net Net-(C1-Pad2): track 0.00 -> 23.8 mm
- net Net-(D2-Pad2): track 37.3 -> 14.8 mm
- net Net-(C2-Pad2): track 0.00 -> 20.3 mm
- net /RESET: track 0.00 -> 9.33 mm
- net Net-(K1-Pad1): track 36.1 -> 28.6 mm
- net Net-(D1-Pad2): track 44.9 -> 48.9 mm
- net Net-(Q2-Pad1): track 5.57 -> 8.81 mm
- added copper zone on B.Cu, net GND
Other:
- board outline added: 73.1 x 86.6 mm
- net class Default: clearance 0.2 -> 0.5
- rule trace_clearance: 0.2 -> 0.5
